Commit message: Add my latest code updates

File: my_arm/urdf/my_arm_2.urdf.xacro (robot description, xacro)
@@ -244,21 +244,21 @@
         <origin xyz="0 0 0" rpy="0 0 0"/>
         <axis xyz="0 0 1"/>
-        <limit lower="0" upper="3.14" effort="10" velocity="1"/>
-  </joint>
-  <joint name="shoulder_joint" type="revolute">
+        <limit lower="-1.57" upper="1.57" effort="10" velocity="1"/>
+  </joint>
+  <joint name="shoulder_joint" type="fixed">
         <parent link="yaw_link"/>
         <child link="shoulder_link"/>
         <origin xyz="0 0.005 0.07" rpy="0 0 0"/>
-        <axis xyz="0 1 0"/>
-        <limit lower="0" upper="3.14" effort="10" velocity="1"/>
-  </joint>
-  <joint name="shoulder_bar_joint" type="fixed">
+        <!-- <axis xyz="0 1 0"/>
+        <limit lower="0" upper="3.14" effort="10" velocity="1"/> -->
+  </joint>
+  <joint name="shoulder_bar_joint" type="revolute">
         <parent link="shoulder_link"/>
         <child link="shoulder_bar_link"/>
         <origin xyz="0 -0.009 0" rpy="0 0 0"/>
         <axis xyz="0 1 0"/>
-        <limit lower="-1.57" upper="1.57" effort="10" velocity="1"/>
-  </joint>
-  <joint name="elbow_joint" type="revolute">
+        <limit lower="0" upper="3.14" effort="10" velocity="1"/>
+  </joint>
+  <joint name="elbow_joint" type="fixed">
         <parent link="shoulder_bar_link"/>
         <child link="elbow_link"/>
@@ -267,12 +267,12 @@
         <limit lower="-3.14" upper="0" effort="10" velocity="1"/>
   </joint>
-  <joint name="elbow_bar_joint" type="fixed">
+  <joint name="elbow_bar_joint" type="revolute">
         <parent link="elbow_link"/>
         <child link="elbow_bar_link"/>
         <origin xyz="0 -0.025 0" rpy="0 -0.2799 0"/>
         <axis xyz="0 1 0"/>
-        <limit lower="-1.57" upper="1.57" effort="10" velocity="1"/>
-  </joint>
-  <joint name="elbow_roll_joint" type="revolute">
+        <limit lower="-3.14" upper="0" effort="10" velocity="1"/>
+  </joint>
+  <joint name="elbow_roll_joint" type="fixed">
         <parent link="elbow_bar_link"/>
         <child link="roll_link"/>
@@ -281,12 +281,12 @@
         <limit lower="-1.57" upper="1.57" effort="10" velocity="1"/>
   </joint>
-  <joint name="elbow_roll_frame_joint" type="fixed">
+  <joint name="elbow_roll_frame_joint" type="revolute">
         <parent link="roll_link"/>
         <child link="roll_pitch_frame_link"/>
         <origin xyz="0 -0.042 0" rpy="0 0 -1.57"/>
-        <axis xyz="0 1 0"/>
-        <limit lower="-1.57" upper="1.57" effort="10" velocity="1"/>
-  </joint>
-  <joint name="wrist_pitch_joint" type="revolute">
+        <axis xyz="1 0 0"/>
+        <limit lower="-1.57" upper="1.57" effort="10" velocity="1"/>
+  </joint>
+  <joint name="wrist_pitch_joint" type="fixed">
         <parent link="roll_pitch_frame_link"/>
         <child link="wrist_pitch_link"/>
@@ -295,10 +295,10 @@
         <limit lower="-1.57" upper="1.57" effort="10" velocity="1"/>
   </joint>
-  <joint name="wrist_pitch_bar_joint" type="fixed">
+  <joint name="wrist_pitch_bar_joint" type="revolute">
         <parent link="wrist_pitch_link"/>
         <child link="wrist_pitch_bar_link"/>
         <origin xyz="0 0.04 0" rpy="0 0 1.57"/>
-        <axis xyz="0 1 0"/>
-        <limit lower="0" upper="3.14" effort="10" velocity="1"/>
+        <axis xyz="1 0 0"/>
+        <limit lower="-1.57" upper="1.57" effort="10" velocity="1"/>
   </joint>
   <joint name="wrist_roll_joint" type="revolute">
@@ -307,5 +307,5 @@
         <origin xyz="-0.015 -0.07 0" rpy="0 0 0"/>
         <axis xyz="0 1 0"/>
-        <limit lower="0" upper="3.14" effort="10" velocity="1"/>
+        <limit lower="-1.57" upper="1.57" effort="10" velocity="1"/>
   </joint>
 </robot>

File: my_arm2_moveit/config/my_arm.ros2_control.xacro (robot description, xacro)
@@ -15,29 +15,29 @@
                 <state_interface name="velocity"/>
             </joint>
-            <joint name="shoulder_joint">
+            <joint name="shoulder_bar_joint">
                 <command_interface name="position"/>
                 <state_interface name="position">
-                  <param name="initial_value">${initial_positions['shoulder_joint']}</param>
+                  <param name="initial_value">${initial_positions['shoulder_bar_joint']}</param>
                 </state_interface>
                 <state_interface name="velocity"/>
             </joint>
-            <joint name="elbow_joint">
+            <joint name="elbow_bar_joint">
                 <command_interface name="position"/>
                 <state_interface name="position">
-                  <param name="initial_value">${initial_positions['elbow_joint']}</param>
+                  <param name="initial_value">${initial_positions['elbow_bar_joint']}</param>
                 </state_interface>
                 <state_interface name="velocity"/>
             </joint>
-            <joint name="elbow_roll_joint">
+            <joint name="elbow_roll_frame_joint">
                 <command_interface name="position"/>
                 <state_interface name="position">
-                  <param name="initial_value">${initial_positions['elbow_roll_joint']}</param>
+                  <param name="initial_value">${initial_positions['elbow_roll_frame_joint']}</param>
                 </state_interface>
                 <state_interface name="velocity"/>
             </joint>
-            <joint name="wrist_pitch_joint">
+            <joint name="wrist_pitch_bar_joint">
                 <command_interface name="position"/>
                 <state_interface name="position">
-                  <param name="initial_value">${initial_positions['wrist_pitch_joint']}</param>
+                  <param name="initial_value">${initial_positions['wrist_pitch_bar_joint']}</param>
                 </state_interface>
                 <state_interface name="velocity"/>
